Commit message: Add camera to the robot

File: urdf/my_robot_static_links.xacro (robot description, xacro)
@@ -61,3 +61,31 @@
         <origin xyz="${bodyOX} ${bodyOY} ${bodyOZ}" rpy="0 0 0"/>
     </joint>
+  <!-- Camera Joint -->
+  <joint name="camera_joint" type="fixed">
+    <axis xyz="0 1 0" />
+    <origin xyz="${bodyLen + bodyLen/2.0} 0 ${tireRad}" rpy="0 0 0"/>
+    <parent link="base_link"/>
+    <child link="camera_link"/>
+  </joint>
+  <!-- Camera -->
+  <link name="camera_link">
+    <collision>
+      <origin xyz="${camera_link/2.0} 0 0" rpy="0 0 0"/>
+      <geometry>
+    <box size="${camera_link} ${camera_link} ${camera_link}"/>
+      </geometry>
+    </collision>
+    <visual>
+      <origin xyz="${camera_link/2.0} 0 0" rpy="0 0 0"/>
+      <geometry>
+    <box size="${camera_link} ${camera_link} ${camera_link}"/>
+      </geometry>
+      <material name="red"/>
+    </visual>
+    <inertial>
+      <mass value="1e-5" />
+      <origin xyz="0 0 0" rpy="0 0 0"/>
+      <inertia ixx="1e-6" ixy="0" ixz="0" iyy="1e-6" iyz="0" izz="1e-6" />
+    </inertial>
+  </link>
 </robot>

File: urdf/my_robot_xacro_defs.xacro (robot description, xacro)
@@ -17,3 +17,5 @@
 <!-- Caster wheel -->
 <xacro:property name="casterRad" value="${(tireDiam - bodyHeight)/2.0}"/>
+<!-- Camera -->
+<xacro:property name="camera_link" value="0.025" /> <!-- Size of square 'camera' box -->
 </robot>
